Commit message: small adjustments

File: urdf/robot4_manipulator.xacro (robot description, xacro)
@@ -159,21 +159,4 @@
   </link>
  <!-- joints definition -->
-<!--
-  <joint name="joint_right_wheel" type="continuous">
-    <origin rpy="0 0 0" xyz="-0.05 0.15 0"/>
-    <child link="link_right_wheel"/>
-    <parent link="link_chassis"/>
-    <axis rpy="0 0 0" xyz="0 1 0"/>
-    <limit effort="10000" velocity="1000"/>
-    <joint_properties damping="1.0" friction="1.0"/>
-  </joint>
-  <joint name="joint_left_wheel" type="continuous">
-    <origin rpy="0 0 0" xyz="-0.05 -0.15 0"/>
-    <child link="link_left_wheel"/>
-    <parent link="link_chassis"/>
-    <axis rpy="0 0 0" xyz="0 1 0"/>
-    <limit effort="10000" velocity="1000"/>
-    <joint_properties damping="1.0" friction="1.0"/>
-  </joint> -->
   <joint name="joint_right_wheel" type="continuous">
     <origin rpy="0 0 0" xyz="0.1 0.15 0"/>
@@ -224,11 +207,4 @@
     <joint_properties damping="1.0" friction="1.0"/>
   </joint>
-  <!--
-  <joint name="joint_manipulator_link1" type="fixed">
-    <origin rpy="0 0 0" xyz="0 0 0.1"/>
-    <child link="manipulator_link1"/>
-    <parent link="manipulator_base"/>
-    <axis rpy="0 0 0" xyz="0 1 0"/>
-  </joint> -->
   <joint name="joint_manipulator_link2" type="revolute">
     <origin rpy="0 0 0" xyz="0 0.05 0.55"/>
@@ -268,31 +244,4 @@
   </joint>
   <!-- laser-scanner definition -->
-  <!--
-   <link name="hokuyo_link">
-	    <collision>
-	      <origin xyz="0 0 0.025" rpy="0 0 0"/>
-	      <geometry>
-		<box size="0.05 0.05 0.05"/>
-	      </geometry>
-	    </collision>
-	    <visual>
-	      <origin xyz="0 0 0.025" rpy="0 0 0"/>
-	      <geometry>
-		<box size="0.05 0.05 0.05"/>
-	      </geometry>
-	      <material name="white"/>
-	    </visual>
-	    <inertial>
-	      <mass value="1e-5" />
-	      <origin xyz="0 0 0" rpy="0 0 0"/>
-	      <inertia ixx="1e-6" ixy="0" ixz="0" iyy="1e-6" iyz="0" izz="1e-6" />
-	    </inertial>
-  </link>
-  <joint name="hokuyo_joint" type="fixed">
-	    <axis xyz="0 1 0" />
-	    <origin xyz="0.28 0 0.05" rpy="0 0 0"/>
-	    <parent link="link_chassis"/>
-	    <child link="hokuyo_link"/>
-  </joint> -->
   <link name="hokuyo_link">
     <inertial>
